File: MDCBoard.brd (EAGLE design)
At the start: 43.9 x 32.6 mm, 200 parts, among them J1 JUMPER-SOLDER, J10 MICROSD-SOCKET, J11 USB-C-RECEPTACLE-KOREANHRO, J2 JUMPER-SOLDER, J3 JUMPER-SOLDER, J4 JUMPER-SOLDER, J5 JST-SM02B-SRSS-TB, J6 JUMPER-SOLDER, J7 JUMPER-SOLDER, J8 JUMPER-SOLDER, Q1 PMOS-NEXPERIA-SOT1220, Q2 PMOS-NEXPERIA-SOT1220, Q3 PMOS-NEXPERIA-SOT1220, Q4 DIODESINC-DMG2305UX, Q5 DIODESINC-DMG2305UX, Q6 DIODESINC-DMG2305UX, Q7 DIODESINC-DMG2305UX, Q8 DIODESINC-DMG2305UX, U1 TI-TPS2116, U10 TI-TPS22919DCK, U11 TI-TPS22919DCK, U12 TI-TPS22919DCK, U13 TI-TPS22919DCK, U14 TI-MSP430FR2422IRHL, U16 TI-TXB0102, U17 PANASONIC-EKMB110711X, U18 LATTICE-ICE40HX4K-BG121, U19 WINBOND-W25Q40EW, U2 DIODESINC-AP7350, U20 NEXPERIA-74LVC1G98-OR-INV-INP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, U21 NEXPERIA-74LVC1G98-BUFFER, U22 ON-AR0330CS1C12SPKA0, U23 ALLIANCE-AS4C8M16MSA-6BIN, U24 STM-STM32F730, U25 DIODESINC-DT1446-04V-7, U26 NEXPERIA-74LVC1G98-INVERTER, U3 NEXPERIA-74LVC1G98-NOR, U4 MICROCHIP-MCP7383X, U5 NEXPERIA-74LVC1G98-INVERTER, U6 EATON-STN101, U7 TI-TPS62A01, U8 TI-TPS62A01, U9 TI-TPS62A01, X1 EPSON-FC-135, X2 SITIME-SIT8021, X3 SITIME-SIT8021

Commit message: 21 airwires
Routing:
- net VDD_BAT: track 26.4 -> 26.9 mm
- net GND: vias 66 -> 67
Changed lines of the file:
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@@
 <layer number="13" name="Route13" color="21" fill="1" visible="no" active="no"/>
 <layer number="14" name="Route14" color="22" fill="1" visible="no" active="no"/>
-<layer number="15" name="Power" color="42" fill="1" visible="no" active="yes"/>
-<layer number="16" name="Bottom" color="1" fill="1" visible="yes" active="yes"/>
-<layer number="17" name="Pads" color="2" fill="1" visible="yes" active="yes"/>
+<layer number="15" name="Power" color="42" fill="1" visible="yes" active="yes"/>
+<layer number="16" name="Bottom" color="1" fill="1" visible="no" active="yes"/>
+<layer number="17" name="Pads" color="2" fill="1" visible="no" active="yes"/>
 <layer number="18" name="Vias" color="2" fill="1" visible="yes" active="yes"/>
 <layer number="19" name="Unrouted" color="6" fill="1" visible="no" active="yes"/>
-<layer number="20" name="Dimension" color="24" fill="1" visible="yes" active="yes"/>
+<layer number="20" name="Dimension" color="24" fill="1" visible="no" active="yes"/>
 <layer number="21" name="tPlace" color="7" fill="1" visible="no" active="yes"/>
-<layer number="22" name="bPlace" color="7" fill="1" visible="yes" active="yes"/>
+<layer number="22" name="bPlace" color="7" fill="1" visible="no" active="yes"/>
 <layer number="23" name="tOrigins" color="15" fill="1" visible="no" active="yes"/>
-<layer number="24" name="bOrigins" color="15" fill="1" visible="yes" active="yes"/>
+<layer number="24" name="bOrigins" color="15" fill="1" visible="no" active="yes"/>
 <layer number="25" name="tNames" color="7" fill="1" visible="no" active="yes"/>
-<layer number="26" name="bNames" color="7" fill="1" visible="yes" active="yes"/>
+<layer number="26" name="bNames" color="7" fill="1" visible="no" active="yes"/>
 <layer number="27" name="tValues" color="7" fill="1" visible="no" active="yes"/>
-<layer number="28" name="bValues" color="7" fill="1" visible="yes" active="yes"/>
+<layer number="28" name="bValues" color="7" fill="1" visible="no" active="yes"/>
 <layer number="29" name="tStop" color="7" fill="3" visible="no" active="yes"/>
-<layer number="30" name="bStop" color="7" fill="6" visible="yes" active="yes"/>
+<layer number="30" name="bStop" color="7" fill="6" visible="no" active="yes"/>
 <layer number="31" name="tCream" color="7" fill="4" visible="no" active="yes"/>
-<layer number="32" name="bCream" color="7" fill="5" visible="yes" active="yes"/>
+<layer number="32" name="bCream" color="7" fill="5" visible="no" active="yes"/>
 <layer number="33" name="tFinish" color="6" fill="3" visible="no" active="yes"/>
-<layer number="34" name="bFinish" color="6" fill="6" visible="yes" active="yes"/>
+<layer number="34" name="bFinish" color="6" fill="6" visible="no" active="yes"/>
 <layer number="35" name="tGlue" color="7" fill="4" visible="no" active="yes"/>
-<layer number="36" name="bGlue" color="7" fill="5" visible="yes" active="yes"/>
+<layer number="36" name="bGlue" color="7" fill="5" visible="no" active="yes"/>
 <layer number="37" name="tTest" color="7" fill="1" visible="no" active="yes"/>
-<layer number="38" name="bTest" color="7" fill="1" visible="yes" active="yes"/>
+<layer number="38" name="bTest" color="7" fill="1" visible="no" active="yes"/>
 <layer number="39" name="tKeepout" color="4" fill="11" visible="no" active="yes"/>
-<layer number="40" name="bKeepout" color="1" fill="11" visible="yes" active="yes"/>
+<layer number="40" name="bKeepout" color="1" fill="11" visible="no" active="yes"/>
 <layer number="41" name="tRestrict" color="4" fill="10" visible="no" active="yes"/>
-<layer number="42" name="bRestrict" color="1" fill="10" visible="yes" active="yes"/>
+<layer number="42" name="bRestrict" color="1" fill="10" visible="no" active="yes"/>
 <layer number="43" name="vRestrict" color="2" fill="10" visible="no" active="yes"/>
 <layer number="44" name="Drills" color="7" fill="1" visible="no" active="yes"/>
@@
 <via x="41.22928125" y="10.149840625" extent="1-16" drill="0.381"/>
 <via x="37.932359375" y="10.302240625" extent="1-16" drill="0.381"/>
+<via x="35.42538125" y="27.802840625" extent="1-16" drill="0.254"/>
+<polygon width="0.127" layer="16" rank="2">
+<vertex x="34.678621875" y="28.702"/>
+<vertex x="34.678621875" y="27.26181875"/>
+<vertex x="36.492178125" y="27.26181875"/>
+<vertex x="36.492178125" y="28.702"/>
+</polygon>
 <wire x1="28.136603125" y1="25.989984375" x2="27.0676375" y2="26.110340625" width="0" layer="19" extent="1-16"/>
 <wire x1="27.192578125" y1="24.960959375" x2="27.0676375" y2="26.110340625" width="0" layer="19" extent="1-16"/>
 <wire x1="28.916" y1="30.917740625" x2="29.6841625" y2="31.831278125" width="0" layer="19" extent="16-16"/>
 <wire x1="29.264359375" y1="28.1267375" x2="28.916" y2="29.437740625" width="0" layer="19" extent="1-16"/>
-<wire x1="35.2861375" y1="28.494596875" x2="35.225" y2="29.97" width="0" layer="19" extent="1-16"/>
 <wire x1="21.93470625" y1="5.83590625" x2="21.030403125" y2="4.67901875" width="0" layer="19" extent="1-16"/>
 <wire x1="19.39933125" y1="2.48265625" x2="18.034" y2="3.81" width="0" layer="19" extent="16-16"/>
@@
 <wire x1="39.34991875" y1="13.9543375" x2="39.34991875" y2="22.290940625" width="0.635" layer="15"/>
 <wire x1="39.34991875" y1="22.290940625" x2="41.037259375" y2="23.97828125" width="0.635" layer="15"/>
-<wire x1="38.01214375" y1="26.95934375" x2="36.3613375" y2="26.95934375" width="0.381" layer="15"/>
-<wire x1="36.3613375" y1="26.95934375" x2="33.104840625" y2="30.215840625" width="0.381" layer="15"/>
+<wire x1="33.104840625" y1="30.215840625" x2="34.87928125" y2="28.4414" width="0.381" layer="15"/>
+<wire x1="34.87928125" y1="28.4414" x2="34.87928125" y2="27.5766375" width="0.381" layer="15"/>
+<wire x1="34.87928125" y1="27.5766375" x2="35.496575" y2="26.95934375" width="0.381" layer="15"/>
+<wire x1="35.496575" y1="26.95934375" x2="38.01214375" y2="26.95934375" width="0.381" layer="15"/>
 </signal>
 <signal name="VDD_B_EN">
@@
 <wire x1="32.821109375" y1="29.285565625" x2="32.821109375" y2="28.64026875" width="0.127" layer="1"/>
 <wire x1="32.821109375" y1="28.64026875" x2="32.6161375" y2="28.435296875" width="0.127" layer="1"/>
-<wire x1="34.438203125" y1="28.445475" x2="36.7687" y2="26.114978125" width="0.127" layer="16"/>
-<wire x1="36.7687" y1="26.114978125" x2="36.7687" y2="24.0687" width="0.127" layer="16"/>
-<wire x1="33.491578125" y1="28.445475" x2="34.438203125" y2="28.445475" width="0.127" layer="16"/>
+<wire x1="36.7687" y1="25.689025" x2="36.7687" y2="24.0687" width="0.127" layer="16"/>
+<wire x1="33.491578125" y1="28.445475" x2="34.268021875" y2="28.445475" width="0.127" layer="16"/>
 <wire x1="32.6161375" y1="28.435296875" x2="33.4814" y2="28.435296875" width="0.127" layer="16"/>
 <wire x1="33.4814" y1="28.435296875" x2="33.491578125" y2="28.445475" width="0.127" layer="16"/>
@@
 <wire x1="39.37" y1="14.732" x2="36.322" y2="11.684" width="0.127" layer="1"/>
 <wire x1="36.322" y1="11.684" x2="29.145734375" y2="11.684" width="0.127" layer="1"/>
+<wire x1="34.268021875" y1="28.445475" x2="34.698940625" y2="28.01455625" width="0.127" layer="16"/>
+<wire x1="34.698940625" y1="28.01455625" x2="34.698940625" y2="27.758784375" width="0.127" layer="16"/>
+<wire x1="34.698940625" y1="27.758784375" x2="36.7687" y2="25.689025" width="0.127" layer="16"/>
 </signal>
 <signal name="N$4">

Commit message: 20 airwires
Parts:
- moved C11 0.13 mm to (29.3, 27.4)
Routing:
- net GND: vias 67 -> 68
Changed lines of the file:
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@@
 <layer number="13" name="Route13" color="21" fill="1" visible="no" active="no"/>
 <layer number="14" name="Route14" color="22" fill="1" visible="no" active="no"/>
-<layer number="15" name="Power" color="42" fill="1" visible="yes" active="yes"/>
-<layer number="16" name="Bottom" color="1" fill="1" visible="no" active="yes"/>
-<layer number="17" name="Pads" color="2" fill="1" visible="no" active="yes"/>
+<layer number="15" name="Power" color="42" fill="1" visible="no" active="yes"/>
+<layer number="16" name="Bottom" color="1" fill="1" visible="yes" active="yes"/>
+<layer number="17" name="Pads" color="2" fill="1" visible="yes" active="yes"/>
 <layer number="18" name="Vias" color="2" fill="1" visible="yes" active="yes"/>
 <layer number="19" name="Unrouted" color="6" fill="1" visible="no" active="yes"/>
-<layer number="20" name="Dimension" color="24" fill="1" visible="no" active="yes"/>
+<layer number="20" name="Dimension" color="24" fill="1" visible="yes" active="yes"/>
 <layer number="21" name="tPlace" color="7" fill="1" visible="no" active="yes"/>
-<layer number="22" name="bPlace" color="7" fill="1" visible="no" active="yes"/>
+<layer number="22" name="bPlace" color="7" fill="1" visible="yes" active="yes"/>
 <layer number="23" name="tOrigins" color="15" fill="1" visible="no" active="yes"/>
-<layer number="24" name="bOrigins" color="15" fill="1" visible="no" active="yes"/>
+<layer number="24" name="bOrigins" color="15" fill="1" visible="yes" active="yes"/>
 <layer number="25" name="tNames" color="7" fill="1" visible="no" active="yes"/>
-<layer number="26" name="bNames" color="7" fill="1" visible="no" active="yes"/>
+<layer number="26" name="bNames" color="7" fill="1" visible="yes" active="yes"/>
 <layer number="27" name="tValues" color="7" fill="1" visible="no" active="yes"/>
-<layer number="28" name="bValues" color="7" fill="1" visible="no" active="yes"/>
+<layer number="28" name="bValues" color="7" fill="1" visible="yes" active="yes"/>
 <layer number="29" name="tStop" color="7" fill="3" visible="no" active="yes"/>
-<layer number="30" name="bStop" color="7" fill="6" visible="no" active="yes"/>
+<layer number="30" name="bStop" color="7" fill="6" visible="yes" active="yes"/>
 <layer number="31" name="tCream" color="7" fill="4" visible="no" active="yes"/>
-<layer number="32" name="bCream" color="7" fill="5" visible="no" active="yes"/>
+<layer number="32" name="bCream" color="7" fill="5" visible="yes" active="yes"/>
 <layer number="33" name="tFinish" color="6" fill="3" visible="no" active="yes"/>
-<layer number="34" name="bFinish" color="6" fill="6" visible="no" active="yes"/>
+<layer number="34" name="bFinish" color="6" fill="6" visible="yes" active="yes"/>
 <layer number="35" name="tGlue" color="7" fill="4" visible="no" active="yes"/>
-<layer number="36" name="bGlue" color="7" fill="5" visible="no" active="yes"/>
+<layer number="36" name="bGlue" color="7" fill="5" visible="yes" active="yes"/>
 <layer number="37" name="tTest" color="7" fill="1" visible="no" active="yes"/>
-<layer number="38" name="bTest" color="7" fill="1" visible="no" active="yes"/>
+<layer number="38" name="bTest" color="7" fill="1" visible="yes" active="yes"/>
 <layer number="39" name="tKeepout" color="4" fill="11" visible="no" active="yes"/>
-<layer number="40" name="bKeepout" color="1" fill="11" visible="no" active="yes"/>
+<layer number="40" name="bKeepout" color="1" fill="11" visible="yes" active="yes"/>
 <layer number="41" name="tRestrict" color="4" fill="10" visible="no" active="yes"/>
-<layer number="42" name="bRestrict" color="1" fill="10" visible="no" active="yes"/>
+<layer number="42" name="bRestrict" color="1" fill="10" visible="yes" active="yes"/>
 <layer number="43" name="vRestrict" color="2" fill="10" visible="no" active="yes"/>
 <layer number="44" name="Drills" color="7" fill="1" visible="no" active="yes"/>
@@
 <attribute name="PN" value="GRM155R61H104KE19D" x="76.101390625" y="40.40700625" size="1.778" layer="28" rot="MR225" display="off"/>
 </element>
-<element name="C11" library="EagleLibrary" package="0805" value="10u" x="29.264359375" y="27.2513375" smashed="yes" rot="R90" grouprefs="_VDD_B_1V8_BUCK">
-<attribute name="MFG" value="Samsung" x="29.264359375" y="27.2513375" size="1.778" layer="27" rot="R90" display="off"/>
-<attribute name="NAME" x="30.991621875" y="27.2809375" size="0.762" layer="25" font="vector" rot="R90"/>
-<attribute name="PN" value="CL21A106KOQNNNE" x="29.264359375" y="27.2513375" size="1.778" layer="27" rot="R90" display="off"/>
+<element name="C11" library="EagleLibrary" package="0805" value="10u" x="29.2735" y="27.3783375" smashed="yes" rot="R90" grouprefs="_VDD_B_1V8_BUCK">
+<attribute name="MFG" value="Samsung" x="29.2735" y="27.3783375" size="1.778" layer="27" rot="R90" display="off"/>
+<attribute name="NAME" x="31.0007625" y="27.4079375" size="0.762" layer="25" font="vector" rot="R90"/>
+<attribute name="PN" value="CL21A106KOQNNNE" x="29.2735" y="27.3783375" size="1.778" layer="27" rot="R90" display="off"/>
 </element>
 <element name="LED3" library="EagleLibrary" package="LED-0603" value="LED" x="41.856178125" y="25.48333125" smashed="yes" rot="MR180">
@@
 <via x="23.910040625" y="29.12871875" extent="1-16" drill="0.381"/>
 <polygon width="0.127" layer="16" thermals="no">
-<vertex x="27.908" y="26.84271875"/>
-<vertex x="27.908" y="25.654"/>
-<vertex x="28.553159375" y="25.654"/>
-<vertex x="28.553159375" y="26.84271875"/>
+<vertex x="27.910540625" y="26.29661875"/>
+<vertex x="27.910540625" y="25.397459375"/>
+<vertex x="29.315159375" y="25.397459375"/>
+<vertex x="29.315159375" y="26.29661875"/>
 </polygon>
 <via x="36.29" y="13.716" extent="1-16" drill="0.381"/>
@@
 <vertex x="36.492178125" y="28.702"/>
 </polygon>
-<wire x1="28.136603125" y1="25.989984375" x2="27.0676375" y2="26.110340625" width="0" layer="19" extent="1-16"/>
+<via x="28.956" y="25.5524" extent="1-16" drill="0.254"/>
 <wire x1="27.192578125" y1="24.960959375" x2="27.0676375" y2="26.110340625" width="0" layer="19" extent="1-16"/>
 <wire x1="28.916" y1="30.917740625" x2="29.6841625" y2="31.831278125" width="0" layer="19" extent="16-16"/>
-<wire x1="29.264359375" y1="28.1267375" x2="28.916" y2="29.437740625" width="0" layer="19" extent="1-16"/>
+<wire x1="29.2735" y1="28.2537375" x2="28.916" y2="29.437740625" width="0" layer="19" extent="1-16"/>
 <wire x1="21.93470625" y1="5.83590625" x2="21.030403125" y2="4.67901875" width="0" layer="19" extent="1-16"/>
 <wire x1="19.39933125" y1="2.48265625" x2="18.034" y2="3.81" width="0" layer="19" extent="16-16"/>

Commit message: 17 airwires
Routing:
- net VDD_B_1V8_IMG_SD: track 89.6 -> 88.9 mm
- net GND: vias 68 -> 69

Commit message: 16 airwires
Routing:
- net GND: vias 69 -> 72
Changed lines of the file:
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@@
 <vertex x="40.64" y="12.499340625"/>
 </polygon>
+<via x="36.819840625" y="22.933659375" extent="1-16" drill="0.381"/>
+<via x="37.592" y="16.764" extent="1-16" drill="0.381"/>
+<via x="38.707059375" y="26.007059375" extent="1-16" drill="0.381"/>
 <wire x1="27.192578125" y1="24.960959375" x2="27.0676375" y2="26.110340625" width="0" layer="19" extent="1-16"/>
 <wire x1="28.916" y1="30.917740625" x2="29.6841625" y2="31.831278125" width="0" layer="19" extent="16-16"/>
@@
 <wire x1="30.695915625" y1="6.69100625" x2="29.8034625" y2="4.99618125" width="0" layer="19" extent="1-1"/>
 <wire x1="28.346978125" y1="9.3113625" x2="29.8810375" y2="8.646903125" width="0" layer="19" extent="1-1"/>
-<wire x1="35.507496875" y1="21.310340625" x2="33.612284375" y2="21.42088125" width="0" layer="19" extent="1-16"/>
 </signal>
 <signal name="ICE_IMG_CLK16MHZ">
@@
 <wire x1="36.7687" y1="24.0687" x2="36.322" y2="23.622" width="0.127" layer="16"/>
 <via x="36.322" y="23.622" extent="1-16" drill="0.254"/>
-<wire x1="36.322" y1="23.622" x2="39.37" y2="20.574" width="0.127" layer="1"/>
+<wire x1="36.322" y1="23.622" x2="36.9036625" y2="23.622" width="0.127" layer="1"/>
+<wire x1="39.37" y1="21.1556625" x2="36.9036625" y2="23.622" width="0.127" layer="1"/>
 <wire x1="29.145734375" y1="11.684" x2="27.696978125" y2="10.23524375" width="0.127" layer="1"/>
 <wire x1="27.696978125" y1="10.23524375" x2="27.696978125" y2="9.3113625" width="0.127" layer="1"/>
-<wire x1="39.37" y1="20.574" x2="39.37" y2="14.732" width="0.127" layer="1"/>
+<wire x1="39.37" y1="21.1556625" x2="39.37" y2="14.732" width="0.127" layer="1"/>
 <wire x1="39.37" y1="14.732" x2="36.322" y2="11.684" width="0.127" layer="1"/>
 <wire x1="36.322" y1="11.684" x2="29.145734375" y2="11.684" width="0.127" layer="1"/>

Commit message: 15 airwires
Changed lines of the file:
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@@
 <grid distance="10" unitdist="mil" unit="mil" style="lines" multiple="1" display="no" altdistance="0.00254" altunitdist="mm" altunit="mil"/>
 <layers>
-<layer number="1" name="Top" color="4" fill="1" visible="no" active="yes"/>
+<layer number="1" name="Top" color="4" fill="1" visible="yes" active="yes"/>
 <layer number="2" name="Ground" color="16" fill="1" visible="no" active="yes"/>
 <layer number="3" name="Route3" color="17" fill="1" visible="no" active="no"/>
@@
 <layer number="13" name="Route13" color="21" fill="1" visible="no" active="no"/>
 <layer number="14" name="Route14" color="22" fill="1" visible="no" active="no"/>
-<layer number="15" name="Power" color="42" fill="1" visible="yes" active="yes"/>
+<layer number="15" name="Power" color="42" fill="1" visible="no" active="yes"/>
 <layer number="16" name="Bottom" color="1" fill="1" visible="no" active="yes"/>
-<layer number="17" name="Pads" color="2" fill="1" visible="no" active="yes"/>
+<layer number="17" name="Pads" color="2" fill="1" visible="yes" active="yes"/>
 <layer number="18" name="Vias" color="2" fill="1" visible="yes" active="yes"/>
 <layer number="19" name="Unrouted" color="6" fill="1" visible="no" active="yes"/>
-<layer number="20" name="Dimension" color="24" fill="1" visible="no" active="yes"/>
-<layer number="21" name="tPlace" color="7" fill="1" visible="no" active="yes"/>
+<layer number="20" name="Dimension" color="24" fill="1" visible="yes" active="yes"/>
+<layer number="21" name="tPlace" color="7" fill="1" visible="yes" active="yes"/>
 <layer number="22" name="bPlace" color="7" fill="1" visible="no" active="yes"/>
-<layer number="23" name="tOrigins" color="15" fill="1" visible="no" active="yes"/>
+<layer number="23" name="tOrigins" color="15" fill="1" visible="yes" active="yes"/>
 <layer number="24" name="bOrigins" color="15" fill="1" visible="no" active="yes"/>
-<layer number="25" name="tNames" color="7" fill="1" visible="no" active="yes"/>
+<layer number="25" name="tNames" color="7" fill="1" visible="yes" active="yes"/>
 <layer number="26" name="bNames" color="7" fill="1" visible="no" active="yes"/>
-<layer number="27" name="tValues" color="7" fill="1" visible="no" active="yes"/>
+<layer number="27" name="tValues" color="7" fill="1" visible="yes" active="yes"/>
 <layer number="28" name="bValues" color="7" fill="1" visible="no" active="yes"/>
-<layer number="29" name="tStop" color="7" fill="3" visible="no" active="yes"/>
+<layer number="29" name="tStop" color="7" fill="3" visible="yes" active="yes"/>
 <layer number="30" name="bStop" color="7" fill="6" visible="no" active="yes"/>
-<layer number="31" name="tCream" color="7" fill="4" visible="no" active="yes"/>
+<layer number="31" name="tCream" color="7" fill="4" visible="yes" active="yes"/>
 <layer number="32" name="bCream" color="7" fill="5" visible="no" active="yes"/>
-<layer number="33" name="tFinish" color="6" fill="3" visible="no" active="yes"/>
+<layer number="33" name="tFinish" color="6" fill="3" visible="yes" active="yes"/>
 <layer number="34" name="bFinish" color="6" fill="6" visible="no" active="yes"/>
-<layer number="35" name="tGlue" color="7" fill="4" visible="no" active="yes"/>
+<layer number="35" name="tGlue" color="7" fill="4" visible="yes" active="yes"/>
 <layer number="36" name="bGlue" color="7" fill="5" visible="no" active="yes"/>
-<layer number="37" name="tTest" color="7" fill="1" visible="no" active="yes"/>
+<layer number="37" name="tTest" color="7" fill="1" visible="yes" active="yes"/>
 <layer number="38" name="bTest" color="7" fill="1" visible="no" active="yes"/>
-<layer number="39" name="tKeepout" color="4" fill="11" visible="no" active="yes"/>
+<layer number="39" name="tKeepout" color="4" fill="11" visible="yes" active="yes"/>
 <layer number="40" name="bKeepout" color="1" fill="11" visible="no" active="yes"/>
-<layer number="41" name="tRestrict" color="4" fill="10" visible="no" active="yes"/>
+<layer number="41" name="tRestrict" color="4" fill="10" visible="yes" active="yes"/>
 <layer number="42" name="bRestrict" color="1" fill="10" visible="no" active="yes"/>
 <layer number="43" name="vRestrict" color="2" fill="10" visible="no" active="yes"/>
@@
 <contactref element="U7" pad="4"/>
 <polygon width="0.127" layer="1" thermals="no">
-<vertex x="28.322021875" y="29.92628125"/>
-<vertex x="26.93771875" y="29.92628125"/>
+<vertex x="28.322021875" y="29.766259375"/>
+<vertex x="27.686" y="29.766259375"/>
+<vertex x="27.686" y="30.988"/>
+<vertex x="26.924" y="30.988"/>
+<vertex x="26.93771875" y="30.97428125"/>
 <vertex x="26.93771875" y="28.64358125"/>
 <vertex x="27.948640625" y="28.64358125"/>
@@
 <vertex x="27.654" y="31.242"/>
 </polygon>
-<wire x1="27.916" y1="30.917740625" x2="27.372425" y2="30.522221875" width="0" layer="19" extent="1-16"/>
 </signal>
 <signal name="VDD_B_1V8">
@@
 <vertex x="25.416259375" y="25.0825"/>
 <vertex x="27.4" y="25.0825"/>
-<vertex x="27.4" y="24.892"/>
-<vertex x="26.8437375" y="24.3357375"/>
-<vertex x="26.226521875" y="24.3357375"/>
-<vertex x="25.73121875" y="24.831040625"/>
-<vertex x="25.416259375" y="24.831040625"/>
+<vertex x="27.4" y="24.235509375"/>
+<vertex x="25.416259375" y="24.235509375"/>
 </polygon>
 <polygon width="0.127" layer="1" thermals="no">
