File: MDCBoard-Rev7.brd (EAGLE design)
At the start: 43.9 x 32.6 mm, 197 parts, among them J1 JUMPER-SOLDER, J10 USB-C-RECEPTACLE-KOREANHRO, J2 JUMPER-SOLDER, J3 JUMPER-SOLDER, J4 JUMPER-SOLDER, J5 BATTERY-HEADER-MOLEX-781710002, J6 JUMPER-SOLDER, J7 JUMPER-SOLDER, J8 JUMPER-SOLDER, J9 MICROSD-SOCKET, Q1 PMOS-NEXPERIA-SOT1220, Q2 PMOS-NEXPERIA-SOT1220, Q3 PMOS-NEXPERIA-SOT1220, Q6 DIODESINC-DMG2305UX, Q7 DIODESINC-DMG2305UX, Q8 DIODESINC-DMG2305UX, SW1 TACTILE-SWITCH, U1 TI-TPS2116, U10 TI-TPS22919DCK, U11 TI-TPS22919DCK, U12 TI-TPS22919DCK, U13 TI-TPS22919DCK, U14 TI-MSP430FR2433IRGE, U16 PANASONIC-EKMB110711X, U17 LATTICE-ICE40HX4K-BG121, U18 WINBOND-W25Q40EW, U19 NEXPERIA-74LVC1G98-OR-INV-INP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, U2 DIODESINC-AP7350, U20 NEXPERIA-74LVC1G98-BUFFER, U21 ON-AR0330CS1C12SPKA0, U22 ALLIANCE-AS4C8M16MSA-6BIN, U23 NEXPERIA-74LVC1G98-INVERTER, U24 STM-STM32F730, U25 DIODESINC-DT1446-04V-7, U26 NEXPERIA-74LVC1G98-MUX-INV-OU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, U27 NEXPERIA-74LVC1G98-MUX-INV-OU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, U28 TI-TPS22919DCK, U3 NEXPERIA-74LVC1G98-NOR, U4 MICROCHIP-MCP7383X, U5 NEXPERIA-NXB0102, U6 EATON-STN101, U7 TI-TPS62A01, U8 TI-TPS62A01, U9 TI-TPS62A01, X1 EPSON-FC-135, X2 SITIME-SIT8021, X3 SITIME-SIT8021

Commit message: Layout progress
Parts:
- removed U26, U27: NEXPERIA-74LVC1G98-MUX-INV-OUTPUT, EagleLibrary:NEXPERIA-SOT363
- removed U28: TI-TPS22919DCK, EagleLibrary:TI-TPS22919DCK
- added LED10, LED9: LEDLED-0603, EagleLibrary:LED-0603
- added Q4, Q5: DIODESINC-DMG2305UX, EagleLibrary:DIODESINC-DMG2305UX
- added R10: 100k, EagleLibrary:0402
- added R44, R45: 1k, EagleLibrary:0402
- added U15: TI-TXB0102, EagleLibrary:TI-TXB0102YZP
- U5: value NEXPERIA-NXB0102 -> NEXPERIA-74LVC1G98-INVERTER; device EagleLibrary:NEXPERIA-NXB0102UN -> EagleLibrary:NEXPERIA-SOT363
- moved U5 30.6 mm to (41.9, 12.1), turned to 90 degrees
- moved LED7 8.74 mm to (40.7, 12.8)
- moved LED8 8.69 mm to (40.7, 13.5)
- moved R42 8.60 mm to (42.7, 12.5)
- moved R43 8.60 mm to (42.7, 13.4)
- moved U4 4.17 mm to (41.7, 21.2)
- moved R7 3.03 mm to (39.9, 19.4)
- moved C25 2.29 mm to (35.6, 28.4), flipped to the bottom, turned to 270 degrees
- moved MH3 1.61 mm to (41.9, 17.4)
- moved R22 1.54 mm to (34.4, 31.6), turned to 180 degrees
- moved R23 0.57 mm to (34.3, 26.8), turned to 180 degrees
- moved C19 0.45 mm to (15.0, 6.30)
- moved R21 0.24 mm to (34.4, 30.8)
Connections:
- removed net BAT_CHRG_EN_: R7.1, U24.R11
- removed net LED_SEL: U14.11, U26.6, U27.6
- removed net LED_SIGNAL: U14.8, U26.1, U27.3
- removed net N$17: R8.1, U28.5, U28.6
- removed net N$5: LED1.A, U26.4
- new net LED_GREEN_: Q4.G, U14.8
- new net LED_RED_: Q5.G, U14.11
- new net N$27: LED10.C, R45.1
- new net N$29: LED9.C, R44.1
- new net N$44: LED1.A, Q4.D
- new net N$9: R8.1, U5.4
- new net STM_LED0: LED10.A, U24.R12
- new net STM_LED1: LED9.A, U24.P12
- net BAT_CHRG_LVL_EN: now also R10.1, U5.1; no longer U28.3
- net BAT_CHRG_STAT: now also U24.R11; no longer U24.R12
- net GND: now also R10.2, R44.2, R45.2, R7.1, U15.B1, U5.2, U5.3, U5.6; no longer U26.2, U27.2, U28.2, U5.B1
- net ICE_MSP_SPI_CLK: now also U15.D2; no longer U5.D2
- net ICE_MSP_SPI_CLK_X: now also U15.A2; no longer U5.A2
- net ICE_MSP_SPI_DATA: now also U15.D1; no longer U5.D1
- net ICE_MSP_SPI_DATA_X: now also U15.A1; no longer U5.A1
- net N$6: now also Q5.D; no longer U27.4
- net VDD_A_3V3: now also Q4.S, Q5.S, U15.B2; no longer U26.3, U26.5, U27.1, U27.5, U5.B2
- net VDD_BAT: now also U5.5; no longer U28.1
- net VDD_B_1V8: now also U15.C1, U15.C2; no longer U5.C1, U5.C2
Routing:
- net LED_SEL: track 69.2 -> 0.00 mm, vias 3 -> 0
- net LED_RED_: track 0.00 -> 67.7 mm, vias 0 -> 3
- net LED_SIGNAL: track 66.6 -> 0.00 mm, vias 3 -> 0
- net LED_GREEN_: track 0.00 -> 63.6 mm, vias 0 -> 3
- net BAT_CHRG_EN_: track 17.0 -> 0.00 mm
- net STM_LED0: track 0.00 -> 16.1 mm
- net STM_LED1: track 0.00 -> 16.0 mm
- net STM_LED2: track 4.73 -> 14.3 mm
- net STM_LED3: track 5.51 -> 14.0 mm
- net BAT_CHRG_STAT: track 20.7 -> 23.9 mm
- net VDD_B_1V8_STM: track 51.8 -> 54.8 mm
- net N$6: track 2.50 -> 4.60 mm
- net N$44: track 0.00 -> 2.02 mm, vias 0 -> 1
- net VDD_BAT: track 25.1 -> 26.9 mm
- net VDD_A_3V3: track 130.8 -> 129.0 mm
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- removed copper zone on layer 1, net N$17
Other:
- outline, holes or cut-outs redrawn
