File: MDCBoard-Rev7.sch (EAGLE design)
At the start: 186 parts, among them J1 JUMPER-SOLDER, J10 MICROSD-SOCKET, J11 USB-C-JACK, J2 JUMPER-SOLDER, J3 JUMPER-SOLDER, J4 JUMPER-SOLDER, J5 JST-PH-2, J6 JUMPER-SOLDER, J7 JUMPER-SOLDER, J8 JUMPER-SOLDER, J9 S-MOUNT-LENS-HOLDER, Q1 PMOS-NEXPERIA-SOT1220, Q2 PMOS-NEXPERIA-SOT1220, Q3 PMOS-NEXPERIA-SOT1220, Q4 PMOS-NEXPERIA-SOT1220, U1 TI-TPS2116, U10 TI-TPS22919DCK, U11 TI-TPS22919DCK, U12 TI-TPS22919DCK, U13 TI-TPS22919DCK, U14 TI-TPS22919DCK, U15 TI-MSP430FR2422IRHL, U16 NXP-NTB0102, U17 NXP-NTB0102, U18 PANASONIC-EKMB110711X, U19 LATTICE-ICE40HX4K-BG121, U2 DIODESINC-AP7350, U20 WINBOND-W25Q40EW, U21 NEXPERIA-74LVC1G98-OR-INV-INP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, U22 NEXPERIA-74LVC1G98-BUFFER, U23 ON-AR0330CS1C12SPKA0, U24 ALLIANCE-AS4C8M16MSA-6BIN, U25 STM-STM32F730, U26 DIODESINC-DT1446-04V-7, U3 NEXPERIA-74LVC1G98-NOR, U4 MICROCHIP-MCP7383X, U5 EATON-STN101, U6 TI-TPS6280XYKAR, U7 TI-TPS6280XYKAR, U8 TI-TPS6280XYKAR, U9 TI-TPS22919DCK, X1 EPSON-FC-135, X2 SITIME-SIT8021, X3 SITIME-SIT8021

Commit message: Layout progress
Parts:
- removed C88: 100n, EagleLibrary:CAPACITOR0402
- removed C89, C90, C91, C92, C93: 2.2u, EagleLibrary:CAPACITOR0402
- removed J11: USB-C-JACK, EagleLibrary:USB-C-JACK
- removed TP2: TEST-POINT, EagleLibrary:TEST-POINT
- removed U26: DIODESINC-DT1446-04V-7, EagleLibrary:DIODESINC-DT1446-04V-7
- added LED10, LED9: LEDLED-0603, EagleLibrary:LEDLED-0603
- added MH1, MH2, MH3: MDC-MOUNT-HOLE, EagleLibrary:MDC-MOUNT-HOLE
- added Q5, Q6, Q7, Q8: DIODESINC-DMG2305UX, EagleLibrary:DIODESINC-DMG2305UX
- added R35: 10k, EagleLibrary:RESISTOR0402
- added R36, R37, R38, R39, R40, R41: 20k, EagleLibrary:RESISTOR0402
- added R42, R43, R44, R45: 1k, EagleLibrary:RESISTOR0402
- added R46: 3k, EagleLibrary:RESISTOR0402
- added R47, R48: 5.1k, EagleLibrary:RESISTOR0402
- added SW1: TACTILE-SWITCH, EagleLibrary:TACTILE-SWITCH
- added TP1: TEST-POINT, EagleLibrary:TEST-POINT
- C11, C7, C9: value 10u -> 22u; PN CL21A106KOQNNNE -> CL21A226MQQNNNG
- C13, C14, C15, C66: value 10u -> 2.2u; device EagleLibrary:CAPACITOR0805 -> EagleLibrary:CAPACITOR0402; MFG Samsung -> Taiyo Yuden; PN CL21A106KOQNNNE -> TMK105CBJ225KV-F
- C17, C18, C21: value 2.2u -> 22p; MFG Taiyo Yuden -> Murata; PN TMK105CBJ225KV-F -> GRM1555C1H220JA01D
- C19, C72, C77: value 2.2u -> 100n; MFG Taiyo Yuden -> Murata; PN TMK105CBJ225KV-F -> GRM155R61H104KE19D
- C20: value 2.2u -> 10u; device EagleLibrary:CAPACITOR0402 -> EagleLibrary:CAPACITOR0805; MFG Taiyo Yuden -> Samsung; PN TMK105CBJ225KV-F -> CL21A106KOQNNNE
- C22, C23, C26: value 22p -> 100n; PN GRM1555C1H220JA01D -> GRM155R61H104KE19D
- C25, C44, C51, C55, C59, C67, C68: value 10u -> 100n; device EagleLibrary:CAPACITOR0805 -> EagleLibrary:CAPACITOR0402; MFG Samsung -> Murata; PN CL21A106KOQNNNE -> GRM155R61H104KE19D
- C28, C30, C32, C40, C64: value 100n -> 10n; MFG Murata -> Samsung; PN GRM155R61H104KE19D -> CL05B103KB5NNNC
- C38, C45, C49, C56, C60, C61: value 100n -> 10u; device EagleLibrary:CAPACITOR0402 -> EagleLibrary:CAPACITOR0805; MFG Murata -> Samsung; PN GRM155R61H104KE19D -> CL21A106KOQNNNE
- C39, C43, C46, C70: value 10n -> 100n; MFG Samsung -> Murata; PN CL05B103KB5NNNC -> GRM155R61H104KE19D
- C41: value 10n -> 10u; device EagleLibrary:CAPACITOR0402 -> EagleLibrary:CAPACITOR0805; PN CL05B103KB5NNNC -> CL21A106KOQNNNE
- C71, C76, C83, C85, C86, C87: value 100n -> 2.2u; MFG Murata -> Taiyo Yuden; PN GRM155R61H104KE19D -> TMK105CBJ225KV-F
- H1: value HEADER-2X2 -> TAGCONNECT-TC2030-NLEDGE; device EagleLibrary:HEADER-2X2 -> EagleLibrary:TAGCONNECT-TC2030-NLEDGE
- J10: value MICROSD-SOCKET -> USB-C-RECEPTACLE-KOREANHRO; device EagleLibrary:MICROSD-SOCKET -> EagleLibrary:USB-C-RECEPTACLE-KOREANHRO
- J5: value JST-PH-2 -> BATTERY-HEADER-MOLEX-781710002; device EagleLibrary:JST-PH-2 -> EagleLibrary:BATTERY-HEADER-MOLEX-781710002; MFG HX (Zhejiang Yueqing Hongxing Elec) -> (none); MFG2 HDGC -> (none); PN HX20007-2AWB -> (none); PN2 HDGC2001WR-S-2P -> (none)
- J9: value S-MOUNT-LENS-HOLDER -> MICROSD-SOCKET; device EagleLibrary:S-MOUNT-LENS-HOLDER -> EagleLibrary:MICROSD-SOCKET; MFG Marshall Electronics -> (none); PN V-LH4 -> (none)
- L1, L2, L3: value 470n -> 1u; MFG Murata -> Samsung; PN DFE201612E-R47M=P2 -> CIGT201610LH1R0MNE
- LED1: value LED -> LEDOSRAM-TOPLED-E1608; device EagleLibrary:LED -> EagleLibrary:LEDOSRAM-TOPLED-E1608; PN KS DELLS1.22-JHKI-1 -> KT DELQS1.12-TIVH-36-S446-10-S
- LED2: value LED -> LEDOSRAM-TOPLED-E1608; device EagleLibrary:LED -> EagleLibrary:LEDOSRAM-TOPLED-E1608; PN KS DELLS1.22-JHKI-1 -> KR DELPS1.22-UHVI-26-H3Q4
- LED3, LED4, LED5, LED6, LED7, LED8: value LED -> LEDLED-0603; device EagleLibrary:LED -> EagleLibrary:LEDLED-0603
- Q4: value PMOS-NEXPERIA-SOT1220 -> DIODESINC-DMG2305UX; device EagleLibrary:PMOS-NEXPERIA-SOT1220 -> EagleLibrary:DIODESINC-DMG2305UX; PN PMPB10UPX -> (none)
- R11: value 86.6k -> 3k; MFG Yageo -> Susumu; PN RC0402FR-0786K6L -> RR0510P-302-D
- R12, R13, R14: value 1.8k -> 100k; MFG TE Connectivity -> Yageo; PN CRGP0402F1K8 -> RC0402FR-07100KL
- R15: value 1.8k -> 200k; MFG TE Connectivity -> Yageo; PN CRGP0402F1K8 -> RC0402FR-13200KL
- R16, R4: value 100 -> 100k; MFG Walsin -> Yageo; PN WR04X1000FQL -> RC0402FR-07100KL
- R17: value 100 -> 365k; PN WR04X1000FQL -> WR04X3653FTL
- R18: value 10k -> 100k; PN RC0402JR-0710KL -> RC0402FR-07100KL
- R21, R22: value 10k -> 100; MFG Yageo -> Walsin; PN RC0402JR-0710KL -> WR04X1000FQL
- R23: value 47k -> 100; PN WR04X473 JTL -> WR04X1000FQL
- R24, R25, R26, R27: value 47k -> 1k; MFG Walsin -> Kamaya; PN WR04X473 JTL -> RGC1/16SC1001DTH
- R28, R29: value 1.8k -> 100; MFG TE Connectivity -> Walsin; PN CRGP0402F1K8 -> WR04X1000FQL
- R3: value 100k -> 10k; PN RC0402FR-07100KL -> RC0402JR-0710KL
- R30, R31: value 1.8k -> 10k; MFG TE Connectivity -> Yageo; PN CRGP0402F1K8 -> RC0402JR-0710KL
- R32: value 3k -> 10k; PN AC0402FR-073KL -> RC0402JR-0710KL
- R33, R34: value 5.1k -> 10k; PN AC0402FR-075K1L -> RC0402JR-0710KL
- R5: value 2.7k -> 100k; MFG Bourns -> Yageo; PN CR0402-JW-272GLF -> RC0402FR-07100KL
- R6: value 100k -> 365k; MFG Yageo -> Walsin; PN RC0402FR-07100KL -> WR04X3653FTL
- R7: value 100k -> 2.7k; MFG Yageo -> Bourns; PN RC0402FR-07100KL -> CR0402-JW-272GLF
- R8: value 300k -> 1k; MFG Walsin -> Kamaya; PN WR04X3003FTL -> RGC1/16SC1001DTH
- U14: value TI-TPS22919DCK -> TI-MSP430FR2433IRGE; device EagleLibrary:TI-TPS22919DCK -> EagleLibrary:TI-MSP430FR2433IRGE
- U15: value TI-MSP430FR2422IRHL -> TI-TXB0102; device EagleLibrary:TI-MSP430FR2422IRHL -> EagleLibrary:TI-TXB0102
- U16: value NXP-NTB0102 -> PANASONIC-EKMB110711X; device EagleLibrary:NXP-NTB0102 -> EagleLibrary:PANASONIC-EKMB110711X; PN (none) -> EKMB1107112
- U17: value NXP-NTB0102 -> LATTICE-ICE40HX4K-BG121; device EagleLibrary:NXP-NTB0102 -> EagleLibrary:LATTICE-ICE40HX4K-BG121
- U18: value PANASONIC-EKMB110711X -> WINBOND-W25Q40EW; device EagleLibrary:PANASONIC-EKMB110711X -> EagleLibrary:WINBOND-W25Q40EW; PN EKMB1107112 -> W25Q40EWUXIE
- U19: value LATTICE-ICE40HX4K-BG121 -> NEXPERIA-74LVC1G98-OR-INV-INPUT; device EagleLibrary:LATTICE-ICE40HX4K-BG121 -> EagleLibrary:NEXPERIA-74LVC1G98-OR-INV-INPUT; PN (none) -> 74LVC1G98GW,125
- U20: value WINBOND-W25Q40EW -> NEXPERIA-74LVC1G98-BUFFER; device EagleLibrary:WINBOND-W25Q40EW -> EagleLibrary:NEXPERIA-74LVC1G98-BUFFER; PN W25Q40EWUXIE -> 74LVC1G98GW,125
- U21: value NEXPERIA-74LVC1G98-OR-INV-INPUT -> ON-AR0330CS1C12SPKA0; device EagleLibrary:NEXPERIA-74LVC1G98-OR-INV-INPUT -> EagleLibrary:ON-AR0330CS1C12SPKA0; PN 74LVC1G98GW,125 -> AR0330CS1C12SPKA0-CR
- U22: value NEXPERIA-74LVC1G98-BUFFER -> ALLIANCE-AS4C8M16MSA-6BIN; device EagleLibrary:NEXPERIA-74LVC1G98-BUFFER -> EagleLibrary:ALLIANCE-AS4C8M16MSA-6BIN; PN 74LVC1G98GW,125 -> (none)
- U23: value ON-AR0330CS1C12SPKA0 -> NEXPERIA-74LVC1G98-INVERTER; device EagleLibrary:ON-AR0330CS1C12SPKA0 -> EagleLibrary:NEXPERIA-74LVC1G98-INVERTER; PN AR0330CS1C12SPKA0-CR -> 74LVC1G98GW,125
- U24: value ALLIANCE-AS4C8M16MSA-6BIN -> STM-STM32F730; device EagleLibrary:ALLIANCE-AS4C8M16MSA-6BIN -> EagleLibrary:STM-STM32F730; PN (none) -> STM32F730I8K6
- U25: value STM-STM32F730 -> DIODESINC-DT1446-04V-7; device EagleLibrary:STM-STM32F730 -> EagleLibrary:DIODESINC-DT1446-04V-7; PN STM32F730I8K6 -> (none)
- U5: value EATON-STN101 -> NEXPERIA-74LVC1G98-INVERTER; device EagleLibrary:EATON-STN101 -> EagleLibrary:NEXPERIA-74LVC1G98-INVERTER; PN STN101050B101 -> 74LVC1G98GW,125
- U6: value TI-TPS6280XYKAR -> EATON-STN101; device EagleLibrary:TI-TPS6280XYKAR -> EagleLibrary:EATON-STN101; PN TPS62801YKAR -> STN101050B101
- U7, U8: value TI-TPS6280XYKAR -> TI-TPS62A01; device EagleLibrary:TI-TPS6280XYKAR -> EagleLibrary:TI-TPS62A01; PN TPS62802YKAR -> (none)
- U9: value TI-TPS22919DCK -> TI-TPS62A01; device EagleLibrary:TI-TPS22919DCK -> EagleLibrary:TI-TPS62A01
Connections:
- removed net BAT_CHRG_LVL_EN_: Q4.G, R6.2, U25E.PE3_A1
- removed net ICE_ST_FLASH_EN: R20.1, U21.IN1, U25F.PF5_K3
- removed net ICE_ST_SPI_CLK: U19E.SPI_SCK_L10, U20.CLK, U25B.PB2_M6
- removed net ICE_ST_SPI_CS_: U19E.SPI_SS_B_K10, U21.IN2, U25E.PE12_R10
- removed net ICE_ST_SPI_D0: U19E.SPI_SI_J9, U20.DO, U25F.PF8_L3
- removed net ICE_ST_SPI_D1: U19C.L7, U20.DI, U25F.PF9_L2
- removed net ICE_ST_SPI_D2: U19C.K6, U25F.PF7_K1
- removed net ICE_ST_SPI_D3: U19C.K7, U25F.PF6_K2
- removed net ICE_ST_SPI_D4: U19C.J7, U25E.PE7_R8
- removed net ICE_ST_SPI_D5: U19C.L8, U25E.PE8_P8
- removed net ICE_ST_SPI_D6: U19E.SPI_SO_K9, U25E.PE9_P9
- removed net ICE_ST_SPI_D7: U19C.J8, U25E.PE10_R9
- removed net ICE_ST_SPI_D_READY: U19C.L5, U25A.PA3_R2
- removed net MSP_RST_X_: U16.A2, U25F.PF0_E2
- removed net MSP_TEST_X: U16.A1, U25I.PI8_D2
- removed net N$14: C23.1, U15C.PA.8/P2.0/UCA0TXD/UCA0SIMO/XOUT, X1.B
- removed net N$17: C22.1, U15C.PA.9/P2.1/UCA0RXD/UCA0SOMI/XIN, X1.A
- removed net N$37: C15.1, J8.1, L3.2, U8.VOS
- removed net N$46: Q4.D, R8.1
- removed net N$5: L1.1, U6.SW
- removed net VDD_B_1V8_IMG: C50.1, C55.1, C56.1, C57.1, C58.1, C59.1, C60.1, C61.1, R21.2, R22.1, U22.VDD, U23A.VDD, U23A.VDD_IO, U9.QOD, U9.VOUT
- removed net VDD_B_1V8_IMG_EN: U15B.PA.0/P1.0/UCB0STE/A0/VEREF+, U9.EN
- removed net VDD_B_1V8_SD: R23.2, R24.2, R25.2, R26.2, R27.2, U12.QOD, U12.VOUT
- removed net VDD_B_2V8_IMG: C51.1, C52.1, C53.1, C54.1, C62.1, C63.1, U10.QOD, U10.VOUT, U23A.VAA, U23A.VAA_PIX, U23A.VDD_MIPI, U23A.VDD_PLL
- removed net VDD_B_2V8_IMG_EN: U10.EN, U15B.PA.2/P1.2/UCB0SIMO/UCB0SDA/SMCLK/A2/VEREF-
- removed net VDD_B_2V8_SD: C68.1, C69.1, J10.VDD, U11.QOD, U11.VOUT
- removed net VDD_B_SD_EN: U11.EN, U12.EN, U15C.PA.B/P2.3/TA1.2/UCB0STE/A5
- new net BAT_CHRG_LVL_EN: R10.1, U14PORT2.PA.E/P2.6/UCA1TXD/UCA1SIMO, U5.IN
- new net BUTTON_SIGNAL_: SW1.1, U14PORT2.PA.D/P2.5/UCA1RXD/UCA1SOMI
- new net ICE_STM_FLASH_EN: R32.1, U19.IN1, U24F.PF5_K3
- new net ICE_STM_SPI_CLK: U17E.SPI_SCK_L10, U18.CLK, U24B.PB2_M6
- new net ICE_STM_SPI_CS_: U17E.SPI_SS_B_K10, U19.IN2, U24E.PE12_R10
- new net ICE_STM_SPI_D0: U17C.L8, U24F.PF8_L3
- new net ICE_STM_SPI_D1: U17C.L7, U24F.PF9_L2
- new net ICE_STM_SPI_D2: U17C.K6, U24F.PF7_K1
- new net ICE_STM_SPI_D3: U17C.K7, U24F.PF6_K2
- new net ICE_STM_SPI_D4: U17E.SPI_SI_J9, U18.DO, U24E.PE7_R8
- new net ICE_STM_SPI_D5: U17E.SPI_SO_K9, U18.DI, U24E.PE8_P8
- new net ICE_STM_SPI_D6: U17C.J7, U24E.PE9_P9
- new net ICE_STM_SPI_D7: U17C.J8, U24E.PE10_R9
- new net ICE_STM_SPI_D_READY: U17C.L5, U24A.PA3_R2
- new net LED_GREEN_: Q4.G, U14PORT1.PA.1/P1.1/UCB0CLK/TA0.1/A1
- new net LED_RED_: Q5.G, U14PORT2.PA.A/P2.2/ACLK
- new net MOTION_EN_: Q6.G, U14PORT3.PB.0/P3.0
- new net MSP_STM_I2C_SCL: R20.1, U14PORT1.PA.3/P1.3/UCB0SOMI/UCB0SCL/MCLK/A3, U24B.PB8_A5
- new net MSP_STM_I2C_SDA: R19.1, U14PORT1.PA.2/P1.2/UCB0SIMO/UCB0SDA/TA0.2/A2/VEREF-, U24B.PB9_B4
- new net MSP_XIN: C17.1, U14PORT2.PA.9/P2.1/XIN, X1.B
- new net MSP_XOUT: C18.1, U14PORT2.PA.8/P2.0/XOUT, X1.A
- new net N$11: Q1.G, R6.1
- new net N$12: R6.2, U3.OUT
- new net N$13: C11.1, J8.1, L3.2, R17.1
- new net N$15: L2.1, U8.SW
- new net N$18: R15.2, R16.1, U8.FB
- new net N$19: C9.1, J7.1, L2.2, R15.1
- new net N$22: L3.1, U9.SW
- new net N$24: L1.1, U7.SW
- new net N$44: LED1.A, Q4.D
- new net N$45: LED1.C, R21.2, R22.2
- new net N$9: R8.1, U5.OUT
- new net SD_PULLUP: Q7.S, Q8.D, R36.2, R37.2, R38.2, R39.2, R40.2, R41.2
- new net SD_PULLUP_1V8_EN_: Q7.G, R35.1, U17C.J3, U23.IN
- new net VDD_B_1V8_IMG_SD: C44.1, C49.1, C50.1, C51.1, C52.1, C53.1, C54.1, C55.1, Q7.D, R33.2, R34.1, U10.QOD, U10.VOUT, U20.VDD, U21A.VDD, U21A.VDD_IO
- new net VDD_B_1V8_IMG_SD_EN: U10.EN, U14PORT1.PA.0/P1.0/UCB0STE/TA0CLK/A0/VEREF+
- new net VDD_B_2V8_IMG_SD: C45.1, C46.1, C47.1, C48.1, C56.1, C57.1, C62.1, C63.1, J9.VDD, Q8.S, R35.2, U11.QOD, U11.VOUT, U21A.VAA, U21A.VAA_PIX, U21A.VDD_MIPI, U21A.VDD_PLL, U23.VDD
- new net VDD_B_2V8_IMG_SD_EN: U11.EN, U14PORT2.PA.B/P2.3
- new net VDD_USB_EN: R3.2, U1.ST, U12.EN, U3.IN1
- net BAT_CHRG_LVL: now also C22.1, R11.1, U14PORT1.PA.7/P1.7/UCA0STE/SMCLK/TDO/A7; no longer R10.1, U25F.PF3_J2
- net BAT_CHRG_STAT: now also U24E.PE15_R11; no longer U25B.PB11_R13
- net GND: now also C44.2, C45.2, C47.2, C48.2, H1.5, J9.GND, MH1.1, MH2.1, MH3.1, R11.2, R16.2, R18.2, R21.1, R22.1, R23.1, R24.2, R25.2, R26.2, R27.2, R4.2, R42.2, R43.2, R44.2, R45.2, R46.1, R47.2, R48.2, R5.2, R7.1, SW1.2, U14POWER.DVSS, U15.GND, U17E.GND_E5, U17E.GND_E6, U17E.GND_E7, U17E.GND_F5, U17E.GND_F6, U17E.GND_F7, U17E.GND_G5, U17E.GND_G6, U17E.GND_G7, U17E.GND_H5, U19.GND, U21A.AGND, U21A.DGND, U21B.SADDR, U21B.TEST, U22A.VSSQ_A3, U22A.VSSQ_B7, U22A.VSSQ_C3, U22A.VSSQ_D7, U22A.VSS_A1, U22A.VSS_E3, U22A.VSS_J1, U23.GND, U24J.BOOT0_D6, U24J.BYPASS_REG_L4, U24L.VREF-_N1, U24L.VSSA_M1, U24L.VSS_D5, U24L.VSS_D7, U24L.VSS_D8, U24L.VSS_D9, U24L.VSS_F10, U24L.VSS_F12, U24L.VSS_F2, U24L.VSS_F6, U24L.VSS_F7, U24L.VSS_F8, U24L.VSS_F9, U24L.VSS_G10, U24L.VSS_G12, U24L.VSS_G2, U24L.VSS_G6, U24L.VSS_G7, U24L.VSS_G8, U24L.VSS_G9, U24L.VSS_H10, U24L.VSS_H12, U24L.VSS_H6, U24L.VSS_H7, U24L.VSS_H8, U24L.VSS_H9, U24L.VSS_J10, U24L.VSS_J6, U24L.VSS_J7, U24L.VSS_J8, U24L.VSS_J9, U24L.VSS_K10, U24L.VSS_K6, U24L.VSS_K7, U24L.VSS_K8, U24L.VSS_K9, U24L.VSS_M8, U24L.VSS_M9, U25.GND, U5.GND, U6.2, U7.PG, U8.PG, U9.PG; no longer C38.2, C39.2, C41.2, C42.2, C88.2, C89.2, C90.2, C91.2, C92.2, C93.2, H1.4, J11.GND, J9.GND1, J9.GND2, R11.1, R13.2, R15.2, R28.2, R29.2, R3.2, R30.2, R31.2, R32.1, R33.2, R34.2, R5.1, R9.2, U14.GND, U15A.GND, U15A.GND_THERMALPAD, U17.GND, U19E.GND_E5, U19E.GND_E6, U19E.GND_E7, U19E.GND_F5, U19E.GND_F6, U19E.GND_F7, U19E.GND_G5, U19E.GND_G6, U19E.GND_G7, U19E.GND_H5, U21.GND, U22.GND, U23A.AGND, U23A.DGND, U23B.SADDR, U23B.TEST, U24A.VSSQ_A3, U24A.VSSQ_B7, U24A.VSSQ_C3, U24A.VSSQ_D7, U24A.VSS_A1, U24A.VSS_E3, U24A.VSS_J1, U25J.BOOT0_D6, U25J.BYPASS_REG_L4, U25L.VREF-_N1, U25L.VSSA_M1, U25L.VSS_D5, U25L.VSS_D7, U25L.VSS_D8, U25L.VSS_D9, U25L.VSS_F10, U25L.VSS_F12, U25L.VSS_F2, U25L.VSS_F6, U25L.VSS_F7, U25L.VSS_F8, U25L.VSS_F9, U25L.VSS_G10, U25L.VSS_G12, U25L.VSS_G2, U25L.VSS_G6, U25L.VSS_G7, U25L.VSS_G8, U25L.VSS_G9, U25L.VSS_H10, U25L.VSS_H12, U25L.VSS_H6, U25L.VSS_H7, U25L.VSS_H8, U25L.VSS_H9, U25L.VSS_J10, U25L.VSS_J6, U25L.VSS_J7, U25L.VSS_J8, U25L.VSS_J9, U25L.VSS_K10, U25L.VSS_K6, U25L.VSS_K7, U25L.VSS_K8, U25L.VSS_K9, U25L.VSS_M8, U25L.VSS_M9, U26.GND, U5.2, U6.GND, U6.MODE, U7.MODE
- net GNDPLL0: now also C41.2, C42.2, U17E.GNDPLL0_L6; no longer C47.2, C48.2, U19E.GNDPLL0_L6
- net GNDPLL1: now also C38.2, C39.2, U17E.GNDPLL1_C5; no longer C44.2, C45.2, U19E.GNDPLL1_C5
- net ICE_CDONE: now also R30.2, U17E.CDONE_K8, U24B.PB1_R4; no longer R18.2, U19E.CDONE_K8, U25B.PB1_R4
- net ICE_CRST_: now also R31.2, U17E.CRESET_B_L9, U24F.PF11_R6; no longer R19.2, U19E.CRESET_B_L9, U25F.PF11_R6
- net ICE_IMG_CLK16MHZ: now also TP1.X, U17B.C11, U20.IN; no longer TP2.X, U19B.C11, U22.IN
- net ICE_LED0: now also LED3.A, U17A.A10; no longer LED4.A, U19A.C9
- net ICE_LED1: now also LED4.A, U17A.A11; no longer LED3.A, U19A.A10
- net ICE_LED2: now also LED5.A, U17A.C9; no longer LED2.A, U19A.A11
- net ICE_LED3: now also LED6.A, U17B.B11; no longer LED1.A, U19B.B11
- net ICE_MSP_SPI_CLK: now also U15.A1, U17D.K2; no longer U17.A2, U19D.K2
- net ICE_MSP_SPI_CLK_X: now also U14PORT1.PA.6/P1.6/UCA0CLK/TA1CLK/TDI/TCLK/A6, U15.B1; no longer U15B.PA.6/P1.6/UCA0CLK/TA0CLK/TDI/TCLK, U17.B2
- net ICE_MSP_SPI_DATA: now also U15.A2, U17C.K3; no longer U17.A1, U19C.K3
- net ICE_MSP_SPI_DATA_X: now also U14PORT1.PA.4/P1.4/UCA0TXD/UCA0SIMO/TA1.2/TCK/A4/VREF+, U14PORT1.PA.5/P1.5/UCA0RXD/UCA0SOMI/TA1.1/TMS/A5, U15.B2; no longer U15B.PA.4/P1.4/UCA0TXD/UCA0SIMO/TA0.1/TCK, U15B.PA.5/P1.5/UCA0RXD/UCA0SOMI/TA0.2/TMS, U17.B1
- net IMG_CLK16MHZ: now also U20.OUT, U21B.EXTCLK; no longer U22.OUT, U23B.EXTCLK
- net IMG_D0: now also U17B.D9, U21B.DOUT0; no longer U19B.E8, U23B.DOUT0
- net IMG_D1: now also U17B.D10, U21B.DOUT1; no longer U19B.D10, U23B.DOUT1
- net IMG_D10: now also U17B.H11, U21B.DOUT10; no longer U19B.H11, U23B.DOUT10
- net IMG_D11: now also U17B.H10, U21B.DOUT11; no longer U19B.H10, U23B.DOUT11
- net IMG_D2: now also U17B.G11, U21B.DOUT2; no longer U19B.G11, U23B.DOUT2
- net IMG_D3: now also U17B.G9, U21B.DOUT3; no longer U19B.G9, U23B.DOUT3
- net IMG_D4: now also U17B.E9, U21B.DOUT4; no longer U19B.E9, U23B.DOUT4
- net IMG_D5: now also U17B.K11, U21B.DOUT5; no longer U19B.K11, U23B.DOUT5
- net IMG_D6: now also U17B.F9, U21B.DOUT6; no longer U19B.F9, U23B.DOUT6
- net IMG_D7: now also U17B.G8, U21B.DOUT7; no longer U19B.G8, U23B.DOUT7
- net IMG_D8: now also U17B.J10, U21B.DOUT8; no longer U19B.J10, U23B.DOUT8
- net IMG_D9: now also U17B.J11, U21B.DOUT9; no longer U19B.J11, U23B.DOUT9
- net IMG_DCLK: now also U17B.F11, U21B.PIXCLK; no longer U19B.F11, U23B.PIXCLK
- net IMG_FV: now also U17B.E11, U21B.FRAME_VALID; no longer U19B.E11, U23B.FRAME_VALID
- net IMG_LV: now also U17B.E10, U21B.LINE_VALID; no longer U19B.E10, U23B.LINE_VALID
- net IMG_RST_: now also R33.1, U17B.D11, U21B.RST_; no longer R21.1, U19B.D11, U23B.RST_
- net IMG_SCLK: now also U17B.G10, U21B.SCLK; no longer U19B.G10, U23B.SCLK
- net IMG_SDATA: now also R34.2, U17B.F10, U21B.SDATA; no longer R22.2, U19B.F10, U23B.SDATA
- net MOTION_SIGNAL: now also U14PORT2.PA.C/P2.4/UCA1CLK, U16.OUT; no longer U15B.PA.3/P1.3/UCB0SOMI/UCB0SCL/MCLK/A3, U18.OUT
- net MSP_RST_: now also C21.1, U14POWER.RST_/NMI/SBWTDIO, U24G.PG12_B8; no longer C26.1, U15A.RST_/NMI/SBWTDIO, U16.B2
- net MSP_TEST: now also U14POWER.TEST/SBWTCK, U24G.PG11_B9; no longer U15A.TEST/SBWTCK, U16.B1
- net N$1: now also R9.2; no longer R7.2
- net N$10: now also R46.2, U24J.OTG_HS_REXT_J15; no longer R32.2, U25J.OTG_HS_REXT_J15
- net N$16: now also LED2.C, R23.2; no longer C9.1, J6.1, L1.2, U6.VOS
- net N$2: now also C82.1, U24K.VCAP_1_M10; no longer C89.1, U25K.VCAP_1_M10
- net N$20: now also R24.1; no longer R14.1
- net N$21: now also R7.2; no longer R5.2
- net N$23: now also LED5.C, R26.1; no longer LED4.C, R15.1
- net N$25: now also C66.1, U24J.VDD12OTGHS_J14; no longer C72.1, U25J.VDD12OTGHS_J14
- net N$26: now also LED4.C, R25.1; no longer LED2.C, R13.1
- net N$27: now also LED10.C, R45.1; no longer LED8.C, R31.1
- net N$28: now also LED6.C, R27.1; no longer LED1.C, R12.1
- net N$29: now also LED9.C, R44.1; no longer LED7.C, R30.1
- net N$30: now also LED8.C, R43.1; no longer LED6.C, R29.1
- net N$31: now also LED7.C, R42.1; no longer LED5.C, R28.1
- net N$32: now also R12.1; no longer R9.1
- net N$33: now also R17.2, R18.1, U9.FB; no longer R4.1, U3.OUT
- net N$34: now also R13.2, R14.1, U7.FB; no longer Q1.G, R4.2
- net N$35: now also J10.CC1, R47.1; no longer J11.CC1, R33.1
- net N$36: now also J10.CC2, R48.1; no longer J11.CC2, R34.1
- net N$38: now also C7.1, J6.1, L1.2, R13.1; no longer R11.2, U8.MODE
- net N$4: now also Q8.G, U23.OUT; no longer L2.1, U7.SW
- net N$40: now also U18.CS_, U19.OUT; no longer U20.CS_, U21.OUT
- net N$42: now also R4.1; no longer R3.1
- net N$54: now also J10.VBUS, U25.IO3, U25.IO4, U25.VDD; no longer J11.VBUS, U26.IO3, U26.IO4, U26.VDD
- net N$6: now also LED2.A, Q5.D; no longer L3.1, U8.SW
- net N$7: now also C83.1, U24K.VCAP_2_F13; no longer C90.1, U25K.VCAP_2_F13
- net N$8: now also C26.1, Q6.D, U16.VDD; no longer C12.1, J7.1, L2.2, U7.VOS
- net RAM_A0: now also U17A.D5, U22B.A0; no longer U19A.D5, U24B.A0
- net RAM_A1: now also U17A.B3, U22B.A1; no longer U19A.B3, U24B.A1
- net RAM_A10: now also U17A.A2, U22B.A10; no longer U19A.A2, U24B.A10
- net RAM_A11: now also U17D.D1, U22B.A11; no longer U19D.D1, U24B.A11
- net RAM_A2: now also U17D.B2, U22B.A2; no longer U19D.B2, U24B.A2
- net RAM_A3: now also U17A.A1, U22B.A3; no longer U19A.A1, U24B.A3
- net RAM_A4: now also U17D.B1, U22B.A4; no longer U19D.B1, U24B.A4
- net RAM_A5: now also U17D.C2, U22B.A5; no longer U19D.C2, U24B.A5
- net RAM_A6: now also U17D.C4, U22B.A6; no longer U19D.C4, U24B.A6
- net RAM_A7: now also U17D.D2, U22B.A7; no longer U19D.D2, U24B.A7
- net RAM_A8: now also U17D.C1, U22B.A8; no longer U19D.C1, U24B.A8
- net RAM_A9: now also U17D.C3, U22B.A9; no longer U19D.C3, U24B.A9
- net RAM_BA0: now also U17A.C7, U22B.BA0; no longer U19A.C7, U24B.BA0
- net RAM_BA1: now also U17A.B4, U22B.BA1; no longer U19A.B4, U24B.BA1
- net RAM_CAS_: now also U17A.D7, U22B.!CAS!; no longer U19A.D7, U24B.!CAS!
- net RAM_CKE: now also U17D.D3, U22B.CKE; no longer U19D.D3, U24B.CKE
- net RAM_CLK: now also U17D.E1, U22B.CLK; no longer U19D.E1, U24B.CLK
- net RAM_CS_: now also U17A.A3, U22B.!CS!; no longer U19A.A3, U24B.!CS!
- net RAM_DQ0: now also U17A.A9, U22B.DQ0; no longer U19A.A9, U24B.DQ0
- net RAM_DQ1: now also U17A.A8, U22B.DQ1; no longer U19A.A8, U24B.DQ1
- net RAM_DQ10: now also U17D.F1, U22B.DQ10; no longer U19D.F1, U24B.DQ10
- net RAM_DQ11: now also U17D.H2, U22B.DQ11; no longer U19D.H2, U24B.DQ11
- net RAM_DQ12: now also U17D.G1, U22B.DQ12; no longer U19D.G1, U24B.DQ12
- net RAM_DQ13: now also U17D.J2, U22B.DQ13; no longer U19D.J2, U24B.DQ13
- net RAM_DQ14: now also U17D.H1, U22B.DQ14; no longer U19D.H1, U24B.DQ14
- net RAM_DQ15: now also U17D.J1, U22B.DQ15; no longer U19D.J1, U24B.DQ15
- net RAM_DQ2: now also U17A.B9, U22B.DQ2; no longer U19A.B9, U24B.DQ2
- net RAM_DQ3: now also U17A.A7, U22B.DQ3; no longer U19A.A7, U24B.DQ3
- net RAM_DQ4: now also U17A.B8, U22B.DQ4; no longer U19A.B8, U24B.DQ4
- net RAM_DQ5: now also U17A.A6, U22B.DQ5; no longer U19A.A6, U24B.DQ5
- net RAM_DQ6: now also U17A.B7, U22B.DQ6; no longer U19A.B7, U24B.DQ6
- net RAM_DQ7: now also U17A.A5, U22B.DQ7; no longer U19A.A5, U24B.DQ7
- net RAM_DQ8: now also U17D.F2, U22B.DQ8; no longer U19D.F2, U24B.DQ8
- net RAM_DQ9: now also U17D.G2, U22B.DQ9; no longer U19D.G2, U24B.DQ9
- net RAM_DQM0: now also U17A.B6, U22B.LDQM; no longer U19A.B6, U24B.LDQM
- net RAM_DQM1: now also U17D.E2, U22B.UDQM; no longer U19D.E2, U24B.UDQM
- net RAM_RAS_: now also U17A.B5, U22B.!RAS!; no longer U19A.B5, U24B.!RAS!
- net RAM_WE_: now also U17A.A4, U22B.!WE!; no longer U19A.A4, U24B.!WE!
- net SD_CLK: now also J9.CLK, R36.1, U17C.L3; no longer J10.CLK, U19C.L3
- net SD_CMD: now also J9.CMD, R37.1, U17C.K4; no longer J10.CMD, R23.1, U19C.K4
- net SD_DAT0: now also J9.DAT0, R38.1, U17C.L2; no longer J10.DAT0, R24.1, U19C.L2
- net SD_DAT1: now also J9.DAT1, R39.1, U17C.L1; no longer J10.DAT1, R25.1, U19C.L1
- net SD_DAT2: now also J9.DAT2, R40.1, U17C.K5; no longer J10.DAT2, R26.1, U19C.K5
- net SD_DAT3: now also J9.DAT3, R41.1, U17C.L4; no longer J10.DAT3, R27.1, U19C.L4
- net STM_CLK16MHZ: now also U24H.PH0_G1; no longer U25H.PH0_G1
- net STM_LED0: now also LED10.A, U24B.PB10_R12; no longer LED8.A, U25D.PD9_P14
- net STM_LED1: now also LED9.A, U24B.PB12_P12; no longer LED7.A, U25D.PD11_N14
- net STM_LED2: now also LED8.A, U24B.PB11_R13; no longer LED6.A, U25D.PD14_M14
- net STM_LED3: now also LED7.A, U24B.PB13_P13; no longer LED5.A, U25D.PD15_L14
- net STM_RST_: now also C65.1, U24J.NRST_J1; no longer C71.1, U25J.NRST_J1
- net STM_SWCLK: now also H1.4, U24A.PA14_A14; no longer H1.2, U25A.PA14_A14
- net STM_SWDIO: now also H1.6, U24A.PA13_A15; no longer H1.1, U25A.PA13_A15
- net USB_D+: now also J10.D+, U24B.PB15_R15, U25.IO2; no longer J11.D+, U25B.PB15_R15, U26.IO2
- net USB_D-: now also J10.D-, U24B.PB14_R14, U25.IO1; no longer J11.D-, U25B.PB14_R14, U26.IO1
- net VCCPLL0: now also C41.1, C42.1, R29.1, U17E.VCCPLL0_J6; no longer C47.1, C48.1, R17.1, U19E.VCCPLL0_J6
- net VCCPLL1: now also C38.1, C39.1, R28.1, U17E.VCCPLL1_C6; no longer C44.1, C45.1, R16.1, U19E.VCCPLL1_C6
- net VDD_A: now also U3.VDD
- net VDD_A_3V3: now also C16.1, C19.1, C20.1, C23.1, Q4.S, Q5.S, Q6.S, U13.VIN, U14POWER.DVCC, U15.VCCB; no longer C21.1, C24.1, C27.1, C29.1, C31.1, U14.VIN, U15A.VDD, U16.VCCB, U17.VCCB, U18.VDD, U3.VDD
- net VDD_B: now also C12.1, U9.EN, U9.VIN; no longer C11.1, C13.1, C14.1, C7.1, U6.EN, U6.VIN
- net VDD_BAT: now also U5.VDD; no longer Q4.S, R6.1
- net VDD_BAT_IN: now also R9.1, U6.1; no longer R7.1, U5.1
- net VDD_B_1V2: now also C27.1, C28.1, C29.1, C30.1, R28.2, R29.2, U17E.VCC_D4, U17E.VCC_D8, U17E.VCC_H4, U17E.VCC_H8; no longer C32.1, C33.1, C34.1, C35.1, R16.2, R17.2, U19E.VCC_D4, U19E.VCC_D8, U19E.VCC_H4, U19E.VCC_H8
- net VDD_B_1V8: now also C13.1, C15.1, C24.1, C31.1, C32.1, C33.1, C34.1, C35.1, C43.1, C58.1, C59.1, C60.1, C61.1, R30.1, R31.1, R32.2, U10.VIN, U15.OE, U15.VCCA, U17E.VCCIO_0_D6, U17E.VCCIO_1_F8, U17E.VCCIO_2_H6, U17E.VCCIO_3_E4, U17E.VCCIO_3_G4, U17E.VCC_SPI_L11, U18.HOLD_, U18.VCC, U18.WP_, U19.VDD, U22A.VDDQ_A7, U22A.VDDQ_B3, U22A.VDDQ_C7, U22A.VDDQ_D3, U22A.VDD_A9, U22A.VDD_E7, U22A.VDD_J9; no longer C16.1, C19.1, C20.1, C30.1, C36.1, C37.1, C38.1, C39.1, C41.1, C46.1, C49.1, C64.1, C65.1, C66.1, C67.1, R18.1, R19.1, R20.2, U13.VIN, U17.OE, U17.VCCA, U19E.VCCIO_0_D6, U19E.VCCIO_1_F8, U19E.VCCIO_2_H6, U19E.VCCIO_3_E4, U19E.VCCIO_3_G4, U19E.VCC_SPI_L11, U20.HOLD_, U20.VCC, U20.WP_, U21.VDD, U24A.VDDQ_A7, U24A.VDDQ_B3, U24A.VDDQ_C7, U24A.VDDQ_D3, U24A.VDD_A9, U24A.VDD_E7, U24A.VDD_J9, U9.VIN
- net VDD_B_1V8_STM: now also C64.1, C67.1, C68.1, C69.1, C71.1, C72.1, C81.1, U12.QOD, U12.VOUT, U13.EN, U24J.PDR_ON_C6, U24K.VBAT_C1, U24K.VDDA_R1, U24K.VDD_C5, U24K.VDD_C7, U24K.VDD_C9, U24K.VDD_F3, U24K.VDD_G13, U24K.VDD_G3, U24K.VDD_J12, U24K.VDD_J13, U24K.VDD_K4, U24K.VDD_N10, U24K.VDD_N8, U24K.VDD_N9, U24K.VREF+_P1; no longer C28.1, C75.1, C76.1, C83.1, C84.1, C85.1, C88.1, C91.1, C92.1, C93.1, U13.QOD, U13.VOUT, U14.EN, U16.OE, U16.VCCA, U25J.PDR_ON_C6, U25K.VBAT_C1, U25K.VDDA_R1, U25K.VDDSDMMC_C8, U25K.VDD_C5, U25K.VDD_C7, U25K.VDD_C9, U25K.VDD_F3, U25K.VDD_G13, U25K.VDD_G3, U25K.VDD_J12, U25K.VDD_J13, U25K.VDD_K4, U25K.VDD_N10, U25K.VDD_N8, U25K.VDD_N9, U25K.VREF+_P1
- net VDD_B_2V8: now also C14.1, C36.1, C37.1, U17E.VPP_2V5_C10; no longer C17.1, C18.1, C42.1, C43.1, U10.VIN, U19E.VPP_2V5_C10
- net VDD_B_3V3_STM: now also C75.1, C76.1, C84.1, C85.1, R19.2, R20.2, U13.QOD, U13.VOUT, U14PORT2.PA.F/P2.7, U24K.VDDSDMMC_C8, U24K.VDDUSB_H13; no longer C81.1, C82.1, U14.QOD, U14.VOUT, U25K.VDDUSB_H13
- net VDD_B_EN: now also R5.1, U14PORT3.PB.1/P3.1/UCA1STE; no longer U15B.PA.1/P1.1/UCB0CLK/ACLK/A1/VREF+
- net VDD_USB: now also R3.1; no longer U13.EN, U3.IN1
- net VDD_USB_IN: now also H1.1; no longer H1.3
Other:
- note added: ""If no external battery is used in the application, it is recommended to connect the VBAT pin to VDD""
- note added: "0.5% resistors to ensure accurate ADC measurements. See math to the right!"
- note added: "Filtering capacitor to filter noise from high-impedance BAT_CHRG_LVL signal."
- note added: "MSP_RST_: MSP430 has an internal 20k-50k pullup on MSP_RST_, so we don't add an external one to save a part."
- note added: "MSP_RST_: The MSP430 datasheet recommends a 1nF capacitor on MSP_RST_, but we don't use that value anywhere else, so we're opting for a much smaller 22pF. (Note that we can't use a larger value because it interferes with Spy-bi-wire comms.) Since the recommended 1nF capacitor is for noise suppression, we should be able to get away with a smaller capacitor, and it hasn't caused issues so far."
- note added: "PFET requirements: - low drain / gate leakage current (Idss, Igss): < 1uA necessary to minimize battery leakage current when system is sleeping - low drain-source resistance (Rdson): < 50mΩ necessary to minimize voltage drop and minimize wasted power"
- note added: "Pulldown prevents a floating input while MSP430 is resetting"
- note added: "Pullup to VDD_USB (TPS2116's VIN1, not its VOUT as shown in the datasheet) to avoid a leakage current that would exist when battery powered. If we did pullup to VDD_A (TPS2116's VOUT), ST would be driven to GND when battery powered, and we'd have a huge leakage current between VDD_A and GND (4.2V/10k = 420uA)."
- note added: "R=100 for 11mA: Vf = 2.2 (3.3-2.2)/100 = 0.011"
- note added: "R=50 for 12mA: Vf = 2.7 (3.3-2.7)/50 = 0.012"
- note added: "Resistor Tolerance Math (Why we need 0.5% resistors) * Formulas KdividerWorstcase = (3*(1-Rtol) / (1*(1+Rtol) + 3*(1-Rtol))) KdividerUndo = 1/(3/(3+1)) = 4/3 VsampleWorstcase = 4.2 Vspan = 4.2-3.6 = 0.6 Err = (KdividerWorstcase * KdividerUndo * VsampleWorstcase - VsampleWorstcase) / Vspan * 1% resistors: Rtol = 0.01 KdividerWorstcase = 0.746 Err = 3.5% * 0.5% resistors: Rtol = 0.005 KdividerWorst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"
- note added: "Resistor limits drive strength to limit inrush current. If the gate resistance is too low, VDD_A will droop and MSP430 will brown out. Originally we used a 10k here, but found that the VDD_BAT drooped ~500mV when the MOSFET turned on. At 365k, VDD_BAT droops ~30mV."
- note added: "SD Pullup Voltage Switching (2.8V <-> 1.8V)"
- note added: "This subcircuit divides VDD_BAT by 1.33, and also prevents the battery drain caused by the voltage divider unless we're connected to USB. It accomplishes the latter by using a buffer to transmit the VDD_BAT voltage based on the BAT_CHRG_LVL_EN signal."
- note added: "Use TXB0102's VCCB for our VDD_A because the datasheet says: "VCCA must not exceed VCCB""
- note added: "Users of BAT_CHRG_LVL should have a capacitor at their input to filter noise."
- note added: "Using 20k pullups so we can hit 400 kHz with open-drain comms: Time to pullup from 0V to 90% of 2.8V: R=20 kΩ C=50 pF t = -R*C*Ln(1-.9) = 2.3 us f = 1/t = 434 kHz"
- note added: "Using a 10k pullup (instead of a 100k) to ensure we override ICE40's builtin ~58k pullup which tries to drive this net to 1.8V."
- note added: "VDDSDMMC Bypass Capacitors"
- note added: "VDD_BAT current consumption must be < 0.6µA for MCP73831T battery detection to work (and therefore BAT_CHRG_STAT to work properly)!! 74LVC1G98GW meets this criteria at room temp, but may not at other temps, so at extreme temps, BAT_CHRG_STAT may report that a battery is present when one isn't."
- note added: "VDD_B_1V8_IMG_SD"
- note added: "VDD_B_2V8_IMG_SD"
- note removed: "Ceff>1uF @ 1.8V bias"
- note removed: "Don't use a pullup resistor on MSP_RST_!! MSP430FR* has an internal 20k-50k pullup, which is already on the low end for correct operation of the level shifter, which requires weak pullups. Adding an external resistor lowers the pullup resistance further (parallel resistors), worsening the level shifter's VOL."
- note removed: "Don't use the recommended 1nF capacitor!! For correct operation of the level shifter, we need a much lower capacitance on MSP_RST, because the level shifter can't drive large capacitive loads. Since the recommended 1nF capacitor is for noise suppression, we should be able to get away with a smaller capacitor."
- note removed: "Limits drive strength to dampen ringing on the PFET's gate"
- note removed: "The MOSFET prevents the battery drain caused by the voltage divider until the time comes that we actually need to measure the battery voltage. When we actually want to sample BAT_CHRG_LVL and accept the ensuing battery drain, STM32 asserts BAT_CHRG_LVL_EN_. STM32 is only running when we're connected to USB and therefore charging the battery, in which case we're not concerned with the small amount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"
- note removed: "Use VCCB side for VDD_A because VCCB has a wider supply voltage range (1.65-5.5 V), giving us more flexibility in the battery voltage."
- note removed: "VDD_B_1V8_IMG"
- note removed: "VDD_B_2V8_IMG"
- note removed: "VDD_B_2V8_SD"
- note removed: "≤ 1% ≤ 200 ppm/°C"
