File: MDCBoard.sch (EAGLE design)
At the start: 197 parts, among them J1 JUMPER-SOLDER, J10 USB-C-RECEPTACLE-KOREANHRO, J2 JUMPER-SOLDER, J3 JUMPER-SOLDER, J4 JUMPER-SOLDER, J5 BATTERY-HEADER-MOLEX-781710002, J6 JUMPER-SOLDER, J7 JUMPER-SOLDER, J8 JUMPER-SOLDER, J9 MICROSD-SOCKET, Q1 PMOS-NEXPERIA-SOT1220, Q2 PMOS-NEXPERIA-SOT1220, Q3 PMOS-NEXPERIA-SOT1220, Q6 DIODESINC-DMG2305UX, Q7 DIODESINC-DMG2305UX, Q8 DIODESINC-DMG2305UX, SW1 TACTILE-SWITCH, U1 TI-TPS2116, U10 TI-TPS22919DCK, U11 TI-TPS22919DCK, U12 TI-TPS22919DCK, U13 TI-TPS22919DCK, U14 TI-MSP430FR2433IRGE, U16 PANASONIC-EKMB110711X, U17 LATTICE-ICE40HX4K-BG121, U18 WINBOND-W25Q40EW, U19 NEXPERIA-74LVC1G98-OR-INV-INP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, U2 DIODESINC-AP7350, U20 NEXPERIA-74LVC1G98-BUFFER, U21 ON-AR0330CS1C12SPKA0, U22 ALLIANCE-AS4C8M16MSA-6BIN, U23 NEXPERIA-74LVC1G98-INVERTER, U24 STM-STM32F730, U25 DIODESINC-DT1446-04V-7, U26 NEXPERIA-74LVC1G98-MUX-INV-OU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, U27 NEXPERIA-74LVC1G98-MUX-INV-OU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, U28 TI-TPS22919DCK, U3 NEXPERIA-74LVC1G98-NOR, U4 MICROCHIP-MCP7383X, U5 NEXPERIA-NXB0102, U6 EATON-STN101, U7 TI-TPS62A01, U8 TI-TPS62A01, U9 TI-TPS62A01, X1 EPSON-FC-135, X2 SITIME-SIT8021, X3 SITIME-SIT8021

Commit message: Layout progress
Parts:
- removed LED3, LED4: LEDLED-0603, EagleLibrary:LEDLED-0603
- removed R24, R25: 1k, EagleLibrary:RESISTOR0402
Connections:
- removed net ICE_LED0: LED3.A, U17A.A10
- removed net ICE_LED1: LED4.A, U17A.A11
- removed net N$20: LED3.C, R24.1
- removed net N$26: LED4.C, R25.1
- net GND: no longer R24.2, R25.2
Changed lines of the file:
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@@
 <attribute name="PN" value="GRM155R61H104KE19D"/>
 </part>
-<part name="LED3" library="EagleLibrary" deviceset="LED" device="LED-0603">
-<attribute name="MFG" value="OSRAM"/>
-<attribute name="PN" value="KS DELLS1.22-JHKI-1"/>
-</part>
-<part name="R24" library="EagleLibrary" deviceset="RESISTOR" device="0402" value="1k">
-<attribute name="MFG" value="Kamaya"/>
-<attribute name="PN" value="RGC1/16SC1001DTH"/>
-</part>
-<part name="LED4" library="EagleLibrary" deviceset="LED" device="LED-0603">
-<attribute name="MFG" value="OSRAM"/>
-<attribute name="PN" value="KS DELLS1.22-JHKI-1"/>
-</part>
-<part name="R25" library="EagleLibrary" deviceset="RESISTOR" device="0402" value="1k">
-<attribute name="MFG" value="Kamaya"/>
-<attribute name="PN" value="RGC1/16SC1001DTH"/>
-</part>
 <part name="LED6" library="EagleLibrary" deviceset="LED" device="LED-0603">
 <attribute name="MFG" value="OSRAM"/>
@@
 <attribute name="PN" x="68.58" y="-101.6" size="1.778" layer="96" display="off"/>
 </instance>
-<instance part="LED3" gate="G$1" x="167.64" y="-33.02" smashed="yes">
-<attribute name="NAME" x="171.196" y="-37.592" size="1.778" layer="95" rot="R90"/>
-<attribute name="MFG" x="167.64" y="-33.02" size="1.778" layer="96" display="off"/>
-<attribute name="PN" x="167.64" y="-33.02" size="1.778" layer="96" display="off"/>
-</instance>
-<instance part="R24" gate="G$1" x="167.64" y="-45.72" smashed="yes" rot="R270">
-<attribute name="NAME" x="168.91" y="-43.18" size="1.778" layer="95"/>
-<attribute name="VALUE" x="168.91" y="-45.72" size="1.778" layer="96"/>
-<attribute name="MFG" x="167.64" y="-45.72" size="1.778" layer="96" rot="R270" display="off"/>
-<attribute name="PN" x="167.64" y="-45.72" size="1.778" layer="96" rot="R270" display="off"/>
-</instance>
-<instance part="LED4" gate="G$1" x="182.88" y="-33.02" smashed="yes">
-<attribute name="NAME" x="186.436" y="-37.592" size="1.778" layer="95" rot="R90"/>
-<attribute name="MFG" x="182.88" y="-33.02" size="1.778" layer="96" display="off"/>
-<attribute name="PN" x="182.88" y="-33.02" size="1.778" layer="96" display="off"/>
-</instance>
-<instance part="R25" gate="G$1" x="182.88" y="-45.72" smashed="yes" rot="R270">
-<attribute name="NAME" x="184.15" y="-43.18" size="1.778" layer="95"/>
-<attribute name="VALUE" x="184.15" y="-45.72" size="1.778" layer="96"/>
-<attribute name="MFG" x="182.88" y="-45.72" size="1.778" layer="96" rot="R270" display="off"/>
-<attribute name="PN" x="182.88" y="-45.72" size="1.778" layer="96" rot="R270" display="off"/>
-</instance>
 <instance part="LED6" gate="G$1" x="213.36" y="-33.02" smashed="yes">
 <attribute name="NAME" x="216.916" y="-37.592" size="1.778" layer="95" rot="R90"/>
@@
 </segment>
 <segment>
-<pinref part="R24" gate="G$1" pin="2"/>
-<wire x1="167.64" y1="-50.8" x2="167.64" y2="-53.34" width="0.1524" layer="91"/>
-<label x="167.64" y="-53.34" size="1.778" layer="95"/>
-</segment>
-<segment>
-<pinref part="R25" gate="G$1" pin="2"/>
-<wire x1="182.88" y1="-50.8" x2="182.88" y2="-53.34" width="0.1524" layer="91"/>
-<label x="182.88" y="-53.34" size="1.778" layer="95"/>
-</segment>
-<segment>
 <pinref part="R27" gate="G$1" pin="2"/>
 <wire x1="213.36" y1="-50.8" x2="213.36" y2="-53.34" width="0.1524" layer="91"/>
@@
 </segment>
 </net>
-<net name="N$20" class="0">
-<segment>
-<pinref part="LED3" gate="G$1" pin="C"/>
-<wire x1="167.64" y1="-38.1" x2="167.64" y2="-40.64" width="0.1524" layer="91"/>
-<pinref part="R24" gate="G$1" pin="1"/>
-</segment>
-</net>
-<net name="N$26" class="0">
-<segment>
-<pinref part="LED4" gate="G$1" pin="C"/>
-<wire x1="182.88" y1="-38.1" x2="182.88" y2="-40.64" width="0.1524" layer="91"/>
-<pinref part="R25" gate="G$1" pin="1"/>
-</segment>
-</net>
 <net name="N$28" class="0">
 <segment>
@@
 </segment>
 </net>
-<net name="ICE_LED1" class="0">
-<segment>
-<pinref part="LED4" gate="G$1" pin="A"/>
-<wire x1="182.88" y1="-30.48" x2="182.88" y2="-27.94" width="0.1524" layer="91"/>
-<label x="182.88" y="-27.94" size="1.778" layer="95"/>
-</segment>
-<segment>
-<pinref part="U17" gate="A" pin="A11"/>
-<wire x1="33.02" y1="40.64" x2="35.56" y2="40.64" width="0.1524" layer="91"/>
-<label x="35.56" y="40.64" size="1.778" layer="95"/>
-</segment>
-</net>
-<net name="ICE_LED0" class="0">
-<segment>
-<pinref part="LED3" gate="G$1" pin="A"/>
-<wire x1="167.64" y1="-30.48" x2="167.64" y2="-27.94" width="0.1524" layer="91"/>
-<label x="167.64" y="-27.94" size="1.778" layer="95"/>
-</segment>
-<segment>
-<pinref part="U17" gate="A" pin="A10"/>
-<wire x1="33.02" y1="43.18" x2="35.56" y2="43.18" width="0.1524" layer="91"/>
-<label x="35.56" y="43.18" size="1.778" layer="95"/>
-</segment>
-</net>
